File: ProgDC.kicad_sch (KiCad schematic)
At the start: 54 parts, among them J1 Conn_02x20_Counter_Clockwise_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, J2 Conn_01x24_Pin, J3 Conn_01x03_Pin, U1 KR580VK28, U2 628512, U3 CPU

Commit message: Fix
Connections:
- net GND: now also D21.9 (A); no longer D21.10 (B)
- net at R15.1 (TOP): now also D21.10 (B); no longer D21.9 (A)
Other:
- moved on the sheet: R15
Changed lines of the file:
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@@
 	)
 	(junction
+		(at 328.93 172.72)
+		(diameter 0)
+		(color 0 0 0 0)
+	)
+	(junction
 		(at 199.39 125.73)
 		(diameter 0)
@@
 	)
 	(junction
-		(at 328.93 167.64)
-		(diameter 0)
-		(color 0 0 0 0)
-	)
-	(junction
 		(at 350.52 116.84)
 		(diameter 0)
@@
 	(wire
 		(pts
-			(xy 330.2 172.72) (xy 330.2 168.91)
-		)
-		(stroke
-			(width 0)
-			(type default)
-		)
-	)
-	(wire
-		(pts
 			(xy 350.52 111.76) (xy 350.52 116.84)
 		)
@@
 	(wire
 		(pts
-			(xy 325.12 171.45) (xy 325.12 168.91)
+			(xy 325.12 171.45) (xy 325.12 167.64)
 		)
 		(stroke
@@
 	(wire
 		(pts
-			(xy 328.93 157.48) (xy 328.93 167.64)
+			(xy 328.93 157.48) (xy 328.93 172.72)
 		)
 		(stroke
@@
 	(wire
 		(pts
-			(xy 330.2 168.91) (xy 325.12 168.91)
-		)
-		(stroke
-			(width 0)
-			(type default)
-		)
-	)
-	(wire
-		(pts
 			(xy 22.86 115.57) (xy 25.4 115.57)
 		)
@@
 	(wire
 		(pts
-			(xy 328.93 167.64) (xy 330.2 167.64)
+			(xy 325.12 167.64) (xy 330.2 167.64)
 		)
 		(stroke
@@
 	(wire
 		(pts
+			(xy 328.93 172.72) (xy 330.2 172.72)
+		)
+		(stroke
+			(width 0)
+			(type default)
+		)
+	)
+	(wire
+		(pts
 			(xy 83.82 166.37) (xy 83.82 176.53)
 		)
@@
 	(symbol
 		(lib_id "Pico-altium-import:root_2_R0125_*")
-		(at 328.93 167.64 270)
+		(at 328.93 172.72 270)
 		(mirror x)
 		(unit 1)
@@
 		(dnp no)
 		(property "Reference" "R15"
-			(at 325.12 174.244 0)
+			(at 325.12 179.324 0)
 			(effects
 				(font
@@
 		)
 		(property "Value" "R0125"
-			(at 331.47 177.546 0)
+			(at 331.47 182.626 0)
 			(effects
 				(font
@@
 		)
 		(property "Footprint" "Resistor_THT:R_Axial_DIN0204_L3.6mm_D1.6mm_P2.54mm_Vertical"
-			(at 328.93 167.64 0)
+			(at 328.93 172.72 0)
 			(effects
 				(font
@@
 		)
 		(property "Datasheet" ""
-			(at 328.93 167.64 0)
+			(at 328.93 172.72 0)
 			(effects
 				(font
@@
 		)
 		(property "Description" "R0125"
-			(at 328.93 167.64 0)
+			(at 328.93 172.72 0)
 			(effects
 				(font
@@
 		)
 		(property "ALTIUM_VALUE" "1K"
-			(at 331.47 173.482 0)
+			(at 331.47 178.562 0)
 			(effects
 				(font
@@
 	(symbol
 		(lib_id "power:+5V")
-		(at 328.93 180.34 0)
+		(at 328.93 185.42 0)
 		(mirror x)
 		(unit 1)
@@
 		(dnp no)
 		(property "Reference" "#PWR07"
-			(at 328.93 176.53 0)
+			(at 328.93 181.61 0)
 			(effects
 				(font
@@
 		)
 		(property "Value" "+5V"
-			(at 328.676 184.404 0)
+			(at 328.676 189.484 0)
 			(effects
 				(font
@@
 		)
 		(property "Footprint" ""
-			(at 328.93 180.34 0)
+			(at 328.93 185.42 0)
 			(effects
 				(font
@@
 		)
 		(property "Datasheet" ""
-			(at 328.93 180.34 0)
+			(at 328.93 185.42 0)
 			(effects
 				(font
@@
 		)
 		(property "Description" "Power symbol creates a global label with name \"+5V\""
-			(at 328.93 180.34 0)
+			(at 328.93 185.42 0)
 			(effects
 				(font

Commit message: Fix bugs
Parts:
- removed R15: R0125, Resistor_THT:R_Axial_DIN0204_L3.6mm_D1.6mm_P2.54mm_Vertical, symbol Pico-altium-import:root_2_R0125_*
- removed VD6, VD7: 1N4148, Diode_THT:D_DO-34_SOD68_P2.54mm_Vertical_AnodeUp, symbol Diode:BAT43
Connections:
- net C800_VI53_2 is gone; now on an unnamed net: D5.13 (A)
- net GND: no longer D21.9 (A)
- net Q0: now also D14.13 (B); no longer D22.9 (A)
- net ~{C800_VI53_2_}: no longer D5.12 (Y)
- net ~{C800_VI53_2}: now also D21.10 (B)
- net at D14.12 (A): now also D21.8 (Y); no longer D22.2 (Y)
- net at D22.8 (Y): no longer D14.13 (B)
- new net: D16.4 (A), D5.12 (Y)
- now unconnected: D22.1 (A)
- no-connect marks 16 -> 20
